File: pcb/golia.sch (EAGLE design)
At the start: 20 parts, among them IC1 xm64a4u, U1 MCP1825S-3302E/DB, X2 EXT

Commit message: Corrected silk screen and measurement layering
Parts:
- E: value (none) -> (none)
Changed lines of the file:
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@@
 <?xml version="1.0" encoding="utf-8"?>
 <!DOCTYPE eagle SYSTEM "eagle.dtd">
-<eagle version="8.1.0">
+<eagle version="8.1.1">
 <drawing>
 <settings>
@@
 <part name="D" library="pinhead" deviceset="PINHD-2X5" device=""/>
 <part name="B" library="pinhead" deviceset="PINHD-2X3" device=""/>
-<part name="E" library="pinhead" deviceset="PINHD-2X3" device=""/>
+<part name="E" library="pinhead" deviceset="PINHD-2X3" device="" value=" "/>
 <part name="+3V1" library="supply1" deviceset="+3V3" device=""/>
 <part name="GND" library="supply1" deviceset="GND" device=""/>
